File: falcoln.brd (EAGLE design)
At the start: 111 x 19.1 mm, 68 parts, among them J1 USB_MINI-B_SMT, Q8010 600mA/40V, U1000 TP4056, U1500 FS312F-G, U1550 FS8205, U2000 MT3608, U2100 M3406, U4000 FM116B, U5000 CH340G, U6000 RICHTEK-RT3000CGQM, U6001 0.1uF, U6100 HDC1080NOPAD, Y5000 12Mhz

Commit message: Missed changes
Parts:
- removed 3V3, ADC, CHPD, DRVA, DRVB, GND, GP0, RST, RX, TX: TPSTP10R, testpad:TP10R
- removed C2104: 47uF, rcl:UD-5X5,8_NICHICON
- removed L2101: 4.7uH, SparkFun-Coils:0805
- removed R1006, R1007, R2103: 1k, rcl:R0603
- removed R1008, R1009: 2k, rcl:R0603
- removed R2102: 4.5k, rcl:R0603
- removed R8007: 100k, rcl:R0603
- removed U2100: M3406, geusebio:SOT23-5
- removed U6000: RICHTEK-RT3000CGQM, geusebio:MDFN-10L_3X3
- removed U6001: 0.1uF, rcl:C0603
- removed U6100: HDC1080NOPAD, geusebio:WSON6_NOPAD
- removed U8000: (no value), ESP8266-ESP12E:ESP8266-ESP12E
- added C8009: 0.1uf, rcl:C0603
- added D2003: (no value), SparkFun-DiscreteSemi:SOD-323
- added U1: ESP-WROOM-32, esp32:ESP-WROOM-32
- L2001: value 10uH -> 22uH; device SparkFun-Coils:0805 -> SparkFun-Coils:SRN6045
- R1001: value 1.2k -> 2k
- R1501: value 1k -> 2k
- R2004: value 7.5k -> 4.5k
- R8005: value 10k -> 400k
- R8006: value 400k -> 100k
- R8020: value 56Ohm -> 1Ohm
- R8021: value 1Ohm -> 56Ohm
- moved LOGO1 150.0 mm to (-15.2, 90.2), turned to 0 degrees
- moved R8004 38.6 mm to (39.1, 2.29), turned to 0 degrees
- moved R8005 33.6 mm to (73.7, 3.56), turned to 270 degrees
- moved R8006 6.23 mm to (71.6, 3.56), turned to 90 degrees
- moved C2006 5.33 mm to (99.6, 9.53)
- moved D2002 4.65 mm to (94.2, 12.2), turned to 180 degrees
- moved R2004 4.02 mm to (82.3, 7.11), turned to 0 degrees
- moved R2005 4.02 mm to (82.3, 5.08), turned to 180 degrees
- moved Q8010 3.59 mm to (76.5, 3.30), turned to 0 degrees
- moved U2000 2.55 mm to (82.5, 10.2), turned to 270 degrees
- moved C1503 1.78 mm to (13.2, 6.60), turned to 180 degrees
- moved Y5000 1.02 mm to (34.5, 9.53)
- moved Y5001 1.02 mm to (34.5, 9.53)
- moved C5002 1.02 mm to (29.0, 2.79)
- moved C5003 1.02 mm to (29.0, 16.3)
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Connections:
- net FS_CS renamed N$11
- net FS_V_BATT renamed N$10
- net N$13 renamed FB
- net OC renamed N$1
- net OD renamed N$8
- net USB_N renamed USB-
- net USB_P renamed USB+
- removed net 5V: C2006.+, C4001.1, D2002.C, R2004.2, U4000.5
- removed net ACC_INT/GPIO15: R8005.2, U6000.P$5, U8000.10
- removed net BATT_SAMP_EN: Q8010.1, U8000.14
- removed net BUCK: D2002.A, L2001.2, U2000.1
- removed net CHRG: R1002.1, R1006.2, U1000.7
- removed net CHRG_3V3: R1006.1, R1008.2, U8000.19
- removed net CS0: U8000.17
- removed net GND_BATT: BT1.GND@1, C1503.2, R1501.1, U1500.6, U1550.3
- removed net MISO: U8000.18
- removed net MOSI: U8000.21
- removed net N$1 (its old number): L2101.1, U2100.3
- removed net SCL/GPIO0: GP0.TP, R8003.2, U$1.4, U5000.13, U6000.P$6, U6100.P$6, U8000.12
- removed net SCLK: U8000.22
- removed net SDA/GPIO4: R8004.2, U6000.P$7, U6100.P$1, U8000.13
- removed net STDBY: R1003.1, R1007.2, U1000.6
- removed net STDBY_3V3: R1007.1, R1009.2, U8000.20
- new net ADC_EN: Q8010.1, U1.8
- new net GPIO0: R8003.2, U$1.4, U1.25, U5000.13
- new net GPIO15: R8004.2
- new net N$19: U1.16
- new net N$20: U1.17
- new net N$21: U1.18
- new net N$22: U1.19
- new net N$23: U1.20
- new net N$24: U1.21
- new net N$25: U1.22
- new net N$26: U1.23
- new net N$27: U1.24
- new net N$3: R1003.1, U1000.6
- new net N$5: BT1.GND@1, C1503.2, U1500.6, U1550.3
- new net SW: D2002.A, D2003.A, L2001.2, U2000.1
- net 3.3V: now also C2006.+, C4001.1, D2002.C, D2003.C, R2004.2, U1.2, U4000.5; no longer 3V3.TP, C2104.+, L2101.2, R2102.2, R8004.1, U6000.P$3, U6000.P$9, U6001.1, U6100.P$5, U8000.8
- net ADC: now also R8005.1, R8006.2, U1.9; no longer ADC.TP, R8006.1, R8007.2, U8000.2
- net BLUE: now also R8020.1, U1.12; no longer R8021.1, U8000.4
- net CH_PD: no longer CHPD.TP, U8000.3
- net DRVA: now also U1.36; no longer DRVA.TP, U8000.7
- net DRVB: now also U1.37; no longer DRVB.TP, U8000.6
- net GND: now also C8009.2, R1501.1, R8004.1, R8006.1, U1.1, U1.15, U1.38, U1.GND; no longer C2104.-, GND.TP, R1008.1, R1009.1, R2103.1, R8005.1, R8007.1, U2100.2, U6000.P$4, U6001.2, U6100.P$2, U8000.9
- net GREEN: now also R8021.1, U1.14; no longer R8020.1, U8000.11
- net N$2: now also R1002.1, U1000.7; no longer R2102.1, R2103.2, U2100.5
- net N$9: now also R8005.2; no longer R8006.2
- net RED: now also U1.13; no longer U8000.5
- net RESET: now also C8009.1, U1.3; no longer RST.TP, U8000.1
- net RX: now also U1.34; no longer RX.TP, U8000.15
- net TX: now also U1.35; no longer TX.TP, U8000.16
- net V_BATT: no longer U2100.1, U2100.4
Routing:
- net SCL/GPIO0: track 97.3 -> 0.00 mm, vias 4 -> 0
- net STDBY_3V3: track 69.0 -> 0.00 mm
- net ACC_INT/GPIO15: track 66.0 -> 0.00 mm, vias 2 -> 0
- net CHRG_3V3: track 65.0 -> 0.00 mm
- net SDA/GPIO4: track 50.6 -> 0.00 mm
- net GREEN: track 83.0 -> 35.5 mm, vias 2 -> 0
- net ADC_EN: track 0.00 -> 43.0 mm, vias 0 -> 2
- net 5V: track 36.1 -> 0.00 mm, vias 2 -> 0
- net GPIO0: track 0.00 -> 26.9 mm, vias 0 -> 3
- net SW: track 0.00 -> 25.0 mm
- net BATT_SAMP_EN: track 24.6 -> 0.00 mm, vias 2 -> 0
- net CH_PD: track 23.2 -> 0.00 mm, vias 1 -> 0
- net DRVA: track 67.0 -> 52.1 mm, vias 2 -> 0
- net RESET: track 55.8 -> 69.5 mm
- net GND_BATT: track 13.3 -> 0.00 mm
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Other:
- board text added: "FALCOLN"
- board text removed: "SUNBIRD"
