File: falcoln.sch (EAGLE design)
At the start: 68 parts, among them J1 USB_MINI-B_SMT, Q8010 600mA/40V, U1000 TP4056, U1500 FS312F-G, U1550 FS8205, U2000 MT3608, U2100 M3406, U4000 FM116B, U5000 CH340G, U6000 RICHTEK-RT3000CGQM, U6001 0.1uF, U6100 HDC1080NOPAD, Y5000 12Mhz

Commit message: Missed changes
Parts:
- removed 3V3, ADC, CHPD, DRVA, DRVB, GND, GP0, RST, RX, TX: TPSTP10R, testpad:TPSTP10R
- removed C2104: 47uF, rcl:CPOL-EUUD-5X5,8
- removed L2101: 4.7uH, SparkFun-Coils:INDUCTOR-0805-3.3UH
- removed R1006, R1007, R2103: 1k, rcl:R-EU_R0603
- removed R1008, R1009: 2k, rcl:R-EU_R0603
- removed R2102: 4.5k, rcl:R-EU_R0603
- removed R8007: 100k, rcl:R-EU_R0603
- removed U2100: M3406, geusebio:M3406
- removed U6000: RICHTEK-RT3000CGQM, geusebio:RICHTEK-RT3000CGQM
- removed U6001: 0.1uF, rcl:C-EUC0603
- removed U6100: HDC1080NOPAD, geusebio:HDC1080NOPAD
- removed U8000: (no value), ESP8266-ESP12E:ESP8266-12EESP8266-ESP12E
- added C8009: 0.1uf, rcl:C-EUC0603
- added D2003: DIODE-SCHOTTKY-PMEG4005EJ, SparkFun-DiscreteSemi:DIODE-SCHOTTKY-PMEG4005EJ
- added U1: ESP-WROOM-32, esp32:ESP-WROOM-32
- L2001: value 10uH -> 22uH; device SparkFun-Coils:INDUCTOR-0805-3.3UH -> SparkFun-Coils:INDUCTOR-SRN6045-33UH
- R1001: value 1.2k -> 2k
- R1501: value 1k -> 2k
- R2004: value 7.5k -> 4.5k
- R8005: value 10k -> 400k
- R8006: value 400k -> 100k
- R8020: value 56Ohm -> 1Ohm
- R8021: value 1Ohm -> 56Ohm
Connections:
- net FS_CS renamed N$11
- net FS_V_BATT renamed N$10
- net N$13 renamed FB
- net OC renamed N$1
- net OD renamed N$8
- net USB_N renamed USB-
- net USB_P renamed USB+
- removed net 5V: C2006.+, C4001.1, D2002.C, R2004.2, U4000.VDD
- removed net ACC_INT/GPIO15: R8005.2, U6000.INT1, U8000.GPIO15
- removed net BATT_SAMP_EN: Q8010.B, U8000.GPIO5
- removed net BUCK: D2002.A, L2001.2, U2000.SW
- removed net CHRG: R1002.1, R1006.2, U1000.CHRG
- removed net CHRG_3V3: R1006.1, R1008.2, U8000.GPIO9
- removed net CS0: U8000.CS0
- removed net GND_BATT: BT1.-, C1503.2, R1501.1, U1500.GND, U1550.S2
- removed net MISO: U8000.MISO
- removed net MOSI: U8000.MOSI
- removed net N$1 (its old number): L2101.1, U2100.SW
- removed net SCL/GPIO0: GP0.PP, R8003.2, U$1.GPIO0, U5000.DTR, U6000.SCL, U6100.SCL, U8000.GPIO0
- removed net SCLK: U8000.SCLK
- removed net SDA/GPIO4: R8004.2, U6000.SDA, U6100.SDA, U8000.GPIO4
- removed net STDBY: R1003.1, R1007.2, U1000.STDBY
- removed net STDBY_3V3: R1007.1, R1009.2, U8000.GPIO10
- new net ADC_EN: Q8010.B, U1.IO32
- new net GPIO0: R8003.2, U$1.GPIO0, U1.IO0, U5000.DTR
- new net GPIO15: R8004.2
- new net N$19: U1.IO13
- new net N$20: U1.SD2
- new net N$21: U1.SD3
- new net N$22: U1.CMD
- new net N$23: U1.CLK
- new net N$24: U1.SDO
- new net N$25: U1.SD1
- new net N$26: U1.IO15
- new net N$27: U1.IO2
- new net N$3: R1003.1, U1000.STDBY
- new net N$5: BT1.-, C1503.2, U1500.GND, U1550.S2
- new net SW: D2002.A, D2003.A, L2001.2, U2000.SW
- net 3.3V: now also C2006.+, C4001.1, D2002.C, D2003.C, R2004.2, U1.3V3, U4000.VDD; no longer 3V3.PP, C2104.+, L2101.2, R2102.2, R8004.1, U6000.VDD, U6000.VDDIO, U6001.1, U6100.VIN, U8000.VCC
- net ADC: now also R8005.1, R8006.2, U1.IO33; no longer ADC.PP, R8006.1, R8007.2, U8000.ADC
- net BLUE: now also R8020.1, U1.IO27; no longer R8021.1, U8000.GPIO16
- net CH_PD: no longer CHPD.PP, U8000.CH_PD
- net DRVA: now also U1.IO22; no longer DRVA.PP, U8000.GPIO13
- net DRVB: now also U1.IO23; no longer DRVB.PP, U8000.GPIO12
- net GND: now also C8009.2, R1501.1, R8004.1, R8006.1, U1.GND, U1.GND@1, U1.GND@15, U1.GND@38; no longer C2104.-, GND.PP, R1008.1, R1009.1, R2103.1, R8005.1, R8007.1, U2100.GND, U6000.GND, U6001.2, U6100.GND, U8000.GND
- net GREEN: now also R8021.1, U1.IO12; no longer R8020.1, U8000.GPIO2
- net N$2: now also R1002.1, U1000.CHRG; no longer R2102.1, R2103.2, U2100.FB
- net N$9: now also R8005.2; no longer R8006.2
- net RED: now also U1.IO14; no longer U8000.GPIO14
- net RESET: now also C8009.1, U1.EN; no longer RST.PP, U8000.REST
- net RX: now also U1.RXD0; no longer RX.PP, U8000.RXD
- net TX: now also U1.TXD0; no longer TX.PP, U8000.TXD
- net V_BATT: no longer U2100.RUN, U2100.VIN
